Commit message: joy node changed

File: fw_description/urdf/fw_rev_04_jay.xacro (robot description, xacro)
@@ -19,8 +19,9 @@
       <origin xyz="0 0 0" rpy="0 0 0"/>
       <geometry>
-        <mesh filename="package://fw_rev_04_description/meshes/bases/Freeway_Hotel_flatdualcam.stl" scale="0.001 0.001 0.001"/>
+        <mesh filename="package://fw_rev_04_description/meshes/bases/Freeway_Hotel_flatdualcam_low_lidar.stl" scale="0.001 0.001 0.001"/>
       </geometry>
       <material name="grey"/>
     </visual>
+<!--
     <collision>
       <origin xyz="-0.15 0 0.51" rpy="0 0 0"/>
@@ -29,5 +30,5 @@
       </geometry>
       <material name="red"/>
-    </collision>
+    </collision> -->
 <!--
     <inertial>
@@ -48,5 +49,5 @@
     <parent link="base_link"/>
     <child link="base_scan"/>
-    <origin xyz="0.0378 0 0.247" rpy="0 0 ${PI}"/>
+    <origin xyz="0.2215 0 0.011" rpy="0 0 ${PI}"/>
   </joint>
   <link name="base_scan">
